Commit message: fix: rdm fix

File: install/robot_ras_ros/share/robot_ras_ros/urdf/camera.xacro (robot description, xacro)
@@ -1 +1,64 @@
-/home/joao-pedro/git/Labyrinth-Hackathon/src/maze_bringup/urdf/camera.xacro
+<?xml version="1.0"?>
+<robot xmlns:xacro="http://www.ros.org/wiki/xacro">
+    <xacro:macro name="camera_mono_macro" params="prefix parent xyz_origem rpy_origem">
+        <xacro:property name="camera_x" value="0.02" />
+        <xacro:property name="camera_y" value="0.05" />
+        <xacro:property name="camera_z" value="0.05" />
+        <xacro:property name="massa_camera" value="0.05" />
+        <link name="${prefix}_camera_link">
+            <visual>
+                <origin xyz="0 0 0" rpy="0 1.57 0"/>
+                <geometry>
+                    <cylinder length="0.05" radius="0.03"/>
+                </geometry>
+                <material name="preto"/>
+            </visual>
+            <collision>
+                <origin xyz="0 0 0" rpy="0 1.57 0"/>
+                <geometry>
+                    <cylinder length="0.05" radius="0.03"/>
+                </geometry>
+            </collision>
+            <inertial>
+                <origin xyz="0 0 0" rpy="0 0 0"/>
+                <mass value="${massa_camera}"/>
+                <inertia ixx="${massa_camera * (camera_y*camera_y + camera_z*camera_z)/12}" ixy="0.0" ixz="0.0" iyy="${massa_camera * (camera_x*camera_x + camera_z*camera_z)/12}" iyz="0.0" izz="${massa_camera * (camera_x*camera_x + camera_y*camera_y)/12}"/>
+            </inertial>
+        </link>
+        <joint name="${prefix}_camera_junta" type="fixed">
+            <parent link="${parent}"/>
+            <child link="${prefix}_camera_link"/>
+            <origin xyz="${xyz_origem}" rpy="${rpy_origem}"/>
+        </joint>
+        <gazebo reference="${prefix}_camera_link">
+            <material>Gazebo/Black</material>
+            <sensor type="camera" name="${prefix}_camera_sensor">
+                <pose>0 0 0 0 0 0</pose>
+                <visualize>false</visualize>
+                <update_rate>90.0</update_rate>
+                <camera name="head">
+                    <horizontal_fov>0.20</horizontal_fov>
+                    <!-- <horizontal_fov>1.047</horizontal_fov> -->
+                    <image>
+                        <width>640</width>
+                        <height>480</height>
+                        <format>R8G8B8</format>
+                    </image>
+                    <clip>
+                        <near>0.01</near>
+                        <far>1.5</far>
+                    </clip>
+                </camera>
+                <plugin name="${prefix}_camera_plugin" filename="libgazebo_ros_camera.so">
+                    <ros>
+                        <namespace>/${prefix}_camera</namespace>
+                        <image_topic>image_raw</image_topic>
+                        <camera_info_topic>camera_info</camera_info_topic>
+                    </ros>
+                    <frame_name>${prefix}_camera_link</frame_name>
+                    <hack_baseline>0.0</hack_baseline>
+                </plugin>
+            </sensor>
+        </gazebo>
+    </xacro:macro>
+</robot>

File: install/robot_ras_ros/share/robot_ras_ros/urdf/chassis.xacro (robot description, xacro)
@@ -1 +1,40 @@
-/home/joao-pedro/git/Labyrinth-Hackathon/src/maze_bringup/urdf/chassis.xacro
+<?xml version="1.0"?>
+<robot xmlns:xacro="http://www.ros.org/wiki/xacro">
+    <xacro:macro name="chassis_macro">
+        <link name="base_link">
+            <visual>
+                <origin xyz="0 0 0" rpy="0 0 0"/>
+                <geometry>
+                    <box size="${comprimento_chassis} ${largura_chassis} ${altura_chassis}"/>
+                </geometry>
+                <material name="azul"/>
+            </visual>
+            <collision>
+                <origin xyz="0 0 0" rpy="0 0 0"/>
+                <geometry>
+                    <box size="${comprimento_chassis} ${largura_chassis} ${altura_chassis}"/>
+                </geometry>
+            </collision>
+            <inertial>
+                <origin xyz="0 0 0" rpy="0 0 0"/>
+                <mass value="${massa_chassis}"/>
+                <inertia ixx="${(1/12) * massa_chassis * (largura_chassis*largura_chassis + altura_chassis*altura_chassis)}" ixy="0.0" ixz="0.0" iyy="${(1/12) * massa_chassis * (comprimento_chassis*comprimento_chassis + altura_chassis*altura_chassis)}" iyz="0.0" izz="${(1/12) * massa_chassis * (comprimento_chassis*comprimento_chassis + largura_chassis*largura_chassis)}"/>
+            </inertial>
+        </link>
+        <gazebo reference="base_link">
+            <material>Gazebo/SkyeBlue</material>
+            <pose>0 0 ${origem_base_link_z_do_chao} 0 0 0</pose>
+        </gazebo>
+        <link name="base_footprint">
+            <inertial>
+                <mass value="0.001"/>
+                <inertia ixx="0.001" ixy="0.0" ixz="0.0" iyy="0.001" iyz="0.0" izz="0.001"/>
+            </inertial>
+        </link>
+        <joint name="base_footprint_joint" type="fixed">
+            <parent link="base_link"/>
+            <child link="base_footprint"/>
+            <origin xyz="0 0 -${origem_base_link_z_do_chao}" rpy="0 0 0"/>
+        </joint>
+    </xacro:macro>
+</robot>

File: install/robot_ras_ros/share/robot_ras_ros/urdf/gazebo_elementos.xacro (robot description, xacro)
@@ -1 +1,32 @@
-/home/joao-pedro/git/Labyrinth-Hackathon/src/maze_bringup/urdf/gazebo_elementos.xacro
+<?xml version="1.0"?>
+<robot xmlns:xacro="http://www.ros.org/wiki/xacro">
+    <xacro:macro name="gazebo_ros2_control_config">
+        <ros2_control name="GazeboSystem" type="system">
+            <hardware>
+                <plugin>gazebo_ros2_control/GazeboSystem</plugin>
+            </hardware>
+            <joint name="left_wheel_joint">
+                <command_interface name="velocity">
+                    <param name="min">-10</param>
+                    <param name="max">10</param>
+                </command_interface>
+                <state_interface name="velocity"/>
+                <state_interface name="position"/>
+            </joint>
+            <joint name="right_wheel_joint">
+                <command_interface name="velocity">
+                    <param name="min">-10</param>
+                    <param name="max">10</param>
+                </command_interface>
+                <state_interface name="velocity"/>
+                <state_interface name="position"/>
+            </joint>
+        </ros2_control>
+        <gazebo>
+            <plugin name="gazebo_ros2_control" filename="libgazebo_ros2_control.so">
+                <robot_param>robot_description</robot_param>
+                <parameters>$(find robot_ras_ros)/params/ros2_control.yaml</parameters>
+            </plugin>
+        </gazebo>
+    </xacro:macro>
+</robot>

File: install/robot_ras_ros/share/robot_ras_ros/urdf/lidar.xacro (robot description, xacro)
@@ -1 +1,68 @@
-/home/joao-pedro/git/Labyrinth-Hackathon/src/maze_bringup/urdf/lidar.xacro
+<?xml version="1.0"?>
+<robot xmlns:xacro="http://www.ros.org/wiki/xacro">
+    <xacro:macro name="lidar_macro" params="prefix parent xyz_origem rpy_origem">
+        <!-- Parâmetros físicos do sensor -->
+        <xacro:property name="tamanho_lidar" value="0.05" />
+        <xacro:property name="massa_lidar" value="0.1" />
+        <link name="${prefix}_lidar_link">
+            <visual>
+                <origin xyz="0 0 0" rpy="0 0 0"/>
+                <geometry>
+                    <cylinder length="0.05" radius="0.03"/>
+                </geometry>
+                <material name="vermelho"/>
+            </visual>
+            <collision>
+                <origin xyz="0 0 0" rpy="0 0 0"/>
+                <geometry>
+                    <cylinder length="0.05" radius="0.03"/>
+                </geometry>
+            </collision>
+            <inertial>
+                <origin xyz="0 0 0" rpy="0 0 0"/>
+                <mass value="${massa_lidar}"/>
+                <inertia ixx="${massa_lidar * (3*0.03*0.03 + 0.05*0.05)/12}" ixy="0.0" ixz="0.0" iyy="${massa_lidar * (3*0.03*0.03 + 0.05*0.05)/12}" iyz="0.0" izz="${massa_lidar * (0.03*0.03)/2}"/>
+            </inertial>
+        </link>
+        <joint name="${prefix}_lidar_junta" type="fixed">
+            <parent link="${parent}"/>
+            <child link="${prefix}_lidar_link"/>
+            <origin xyz="${xyz_origem}" rpy="${rpy_origem}"/>
+        </joint>
+        <gazebo reference="${prefix}_lidar_link">
+            <material>Gazebo/Red</material>
+            <sensor type="ray" name="${prefix}_range_sensor">
+                <pose>0 0 0 0 0 0</pose>
+                <visualize>true</visualize>
+                <update_rate>100</update_rate>
+                <ray>
+                    <scan>
+                        <horizontal>
+                            <samples>1</samples>
+                            <resolution>1.0</resolution>
+                            <min_angle>0</min_angle>
+                            <max_angle>0</max_angle>
+                        </horizontal>
+                    </scan>
+                    <range>
+                        <min>0.05</min>
+                        <max>100.0</max>
+                        <resolution>0.01</resolution>
+                    </range>
+                    <noise>
+                        <type>gaussian</type>
+                        <mean>0.0</mean>
+                        <stddev>0.00</stddev>
+                    </noise>
+                </ray>
+                <plugin name="${prefix}_range_plugin" filename="libgazebo_ros_ray_sensor.so">
+                    <ros>
+                        <remapping>~/out:=sensor_range/${prefix}</remapping>
+                    </ros>
+                    <frame_name>${prefix}_lidar_link</frame_name>
+                    <output_type>sensor_msgs/Range</output_type>
+                </plugin>
+            </sensor>
+        </gazebo>
+    </xacro:macro>
+</robot>

File: install/robot_ras_ros/share/robot_ras_ros/urdf/materiais.xacro (robot description, xacro)
@@ -1 +1,18 @@
-/home/joao-pedro/git/Labyrinth-Hackathon/src/maze_bringup/urdf/materiais.xacro
+<?xml version="1.0"?>
+<robot xmlns:xacro="http://www.ros.org/wiki/xacro">
+  <material name="preto">
+    <color rgba="0.1 0.1 0.1 1.0"/>
+  </material>
+  <material name="azul">
+    <color rgba="0.2 0.2 0.8 1.0"/>
+  </material>
+  <material name="branco">
+    <color rgba="0.9 0.9 0.9 1.0"/>
+  </material>
+  <material name="vermelho">
+    <color rgba="0.8 0.1 0.1 1.0"/>
+  </material>
+  <material name="cinza_claro">
+    <color rgba="0.75 0.75 0.75 1.0"/>
+  </material>
+</robot>

File: install/robot_ras_ros/share/robot_ras_ros/urdf/propriedades.xacro (robot description, xacro)
@@ -1 +1,30 @@
-/home/joao-pedro/git/Labyrinth-Hackathon/src/maze_bringup/urdf/propriedades.xacro
+<?xml version="1.0"?>
+<robot xmlns:xacro="http://www.ros.org/wiki/xacro">
+  <xacro:property name="PI" value="3.1415926535897931"/>
+  <xacro:property name="fator_escala" value="0.8" />
+  <xacro:property name="fator_escala_cubico" value="${fator_escala * fator_escala * fator_escala}" />
+  <xacro:property name="altura_total_robo" value="${0.5 * fator_escala}" />
+  <xacro:property name="largura_total_robo" value="${0.9 * fator_escala}" />
+  <xacro:property name="comprimento_total_robo" value="${1.0 * fator_escala}" />
+  <xacro:property name="comprimento_chassis" value="${1.0 * fator_escala}" />
+  <xacro:property name="largura_chassis" value="${largura_total_robo - 2 * espessura_roda}" />
+  <xacro:property name="altura_chassis" value="${0.5 * fator_escala}" />
+  <xacro:property name="massa_chassis" value="${15.0 * fator_escala_cubico}" />
+  <xacro:property name="folga_chao" value="${0.1 * fator_escala}" />
+  <xacro:property name="origem_base_link_z_do_chao" value="${folga_chao + altura_chassis/2}" />
+  <xacro:property name="raio_roda" value="${0.25 * fator_escala}" />
+  <xacro:property name="espessura_roda" value="${0.05 * fator_escala}" />
+  <xacro:property name="massa_roda" value="${1.0 * fator_escala_cubico}" />
+  <xacro:property name="pos_x_junta_roda" value="0.0" />
+  <xacro:property name="pos_y_junta_roda" value="${largura_chassis/2 + espessura_roda/2}" />
+  <xacro:property name="pos_z_junta_roda" value="${raio_roda - origem_base_link_z_do_chao}" />
+  <xacro:property name="raio_roda_boba" value="${0.1 * fator_escala}" />
+  <xacro:property name="massa_roda_boba" value="${0.5 * fator_escala_cubico}" />
+  <xacro:property name="pos_x_roda_boba" value="${comprimento_chassis/2 - raio_roda_boba - (0.02 * fator_escala)}" />
+  <xacro:property name="pos_z_roda_boba" value="${raio_roda_boba - origem_base_link_z_do_chao}" />
+  <xacro:property name="tamanho_lidar" value="${0.05 * fator_escala}" />
+  <xacro:property name="massa_lidar" value="${0.1 * fator_escala_cubico}" />
+  <xacro:property name="pos_z_lidar" value="${altura_chassis/2 - tamanho_lidar}" />
+  <xacro:property name="pos_xy_borda_lidar_frente_tras" value="${comprimento_chassis/2 - tamanho_lidar/4}" />
+  <xacro:property name="pos_xy_borda_lidar_lados" value="${largura_chassis/2 - tamanho_lidar/4}" />
+</robot>

File: install/robot_ras_ros/share/robot_ras_ros/urdf/robot.urdf.xacro (robot description, xacro)
@@ -1 +1,23 @@
-/home/joao-pedro/git/Labyrinth-Hackathon/src/maze_bringup/urdf/robot.urdf.xacro
+<?xml version="1.0"?>
+<robot name="robot_diff"
+    xmlns:xacro="http://www.ros.org/wiki/xacro">
+    <xacro:include filename="propriedades.xacro"/>
+    <xacro:include filename="materiais.xacro"/>
+    <xacro:include filename="chassis.xacro"/>
+    <xacro:include filename="roda.xacro"/>
+    <xacro:include filename="roda_boba.xacro"/>
+    <xacro:include filename="lidar.xacro"/>
+    <xacro:include filename="camera.xacro"/>
+    <xacro:include filename="gazebo_elementos.xacro"/>
+    <xacro:chassis_macro/>
+    <xacro:roda_macro prefix="left" parent="base_link" y_espelho="1"/>
+    <xacro:roda_macro prefix="right" parent="base_link" y_espelho="-1"/>
+    <xacro:roda_boba_macro prefix="front" parent="base_link" x_offset="${pos_x_roda_boba}" y_offset="0" z_offset="${pos_z_roda_boba}"/>
+    <xacro:roda_boba_macro prefix="rear" parent="base_link" x_offset="${-pos_x_roda_boba}" y_offset="0" z_offset="${pos_z_roda_boba}"/>
+    <xacro:lidar_macro prefix="front" parent="base_link" xyz_origem="${pos_xy_borda_lidar_frente_tras} 0 ${pos_z_lidar}" rpy_origem="0 0 0"/>
+    <xacro:lidar_macro prefix="rear" parent="base_link" xyz_origem="-${pos_xy_borda_lidar_frente_tras} 0 ${pos_z_lidar}" rpy_origem="0 0 ${PI}"/>
+    <xacro:lidar_macro prefix="left" parent="base_link" xyz_origem="0.25 ${pos_xy_borda_lidar_lados} ${pos_z_lidar}" rpy_origem="0 0 ${PI/2}"/>
+    <xacro:lidar_macro prefix="right" parent="base_link" xyz_origem="0.25 -${pos_xy_borda_lidar_lados} ${pos_z_lidar}" rpy_origem="0 0 -${PI/2}"/>
+    <xacro:camera_mono_macro prefix="frente" parent="base_link" xyz_origem="${pos_xy_borda_lidar_frente_tras} 0 ${pos_z_lidar - 0.2}" rpy_origem="0 0 0" />
+    <xacro:gazebo_ros2_control_config/>
+</robot>

File: install/robot_ras_ros/share/robot_ras_ros/urdf/roda.xacro (robot description, xacro)
@@ -1 +1,50 @@
-/home/joao-pedro/git/Labyrinth-Hackathon/src/maze_bringup/urdf/roda.xacro
+<?xml version="1.0"?>
+<robot xmlns:xacro="http://www.ros.org/wiki/xacro">
+    <xacro:macro name="roda_macro" params="prefix parent y_espelho">
+        <link name="${prefix}_roda_link">
+            <visual>
+                <origin xyz="0 0 0" rpy="${PI/2} 0 0"/>
+                <geometry>
+                    <cylinder radius="${raio_roda}" length="${espessura_roda}"/>
+                </geometry>
+                <material name="preto"/>
+            </visual>
+            <collision>
+                <origin xyz="0 0 0" rpy="${PI/2} 0 0"/>
+                <geometry>
+                    <cylinder radius="${raio_roda}" length="${espessura_roda}"/>
+                </geometry>
+            </collision>
+            <inertial>
+                <origin xyz="0 0 0" rpy="${PI/2} 0 0"/>
+                <mass value="${massa_roda}"/>
+                <inertia ixx="${(1/12) * massa_roda * (3*raio_roda*raio_roda + espessura_roda*espessura_roda)}" ixy="0.0" ixz="0.0" iyy="${(1/12) * massa_roda * (3*raio_roda*raio_roda + espessura_roda*espessura_roda)}" iyz="0.0" izz="${(1/2) * massa_roda * (raio_roda*raio_roda)}"/>
+            </inertial>
+        </link>
+        <joint name="${prefix}_wheel_joint" type="continuous">
+            <parent link="${parent}"/>
+            <child link="${prefix}_roda_link"/>
+            <origin xyz="${pos_x_junta_roda} ${y_espelho * pos_y_junta_roda} ${pos_z_junta_roda}" rpy="0 0 0"/>
+            <axis xyz="0 1 0"/>
+            <limit effort="100" velocity="100"/>
+        </joint>
+        <gazebo reference="${prefix}_roda_link">
+            <material>Gazebo/DarkGrey</material>
+            <mu1>0.8</mu1>
+            <mu2>0.8</mu2>
+            <kp>1000000.0</kp>
+            <kd>100.0</kd>
+            <minDepth>0.001</minDepth>
+            <maxVel>0.1</maxVel>
+            <fdir1>1 0 0</fdir1>
+        </gazebo>
+        <transmission name="${prefix}_roda_transmissao">
+            <type>transmission_interface/SimpleTransmission</type>
+            <joint name="${prefix}_wheel_joint">
+            </joint>
+            <actuator name="${prefix}_roda_motor">
+                <mechanicalReduction>1</mechanicalReduction>
+            </actuator>
+        </transmission>
+    </xacro:macro>
+</robot>

File: install/robot_ras_ros/share/robot_ras_ros/urdf/roda_boba.xacro (robot description, xacro)
@@ -1 +1,58 @@
-/home/joao-pedro/git/Labyrinth-Hackathon/src/maze_bringup/urdf/roda_boba.xacro
+<?xml version="1.0"?>
+<robot xmlns:xacro="http://www.ros.org/wiki/xacro">
+    <xacro:macro name="roda_boba_macro" params="prefix parent x_offset y_offset z_offset">
+        <link name="${prefix}_roda_boba_link">
+            <visual>
+                <origin xyz="0 0 0" rpy="0 0 0"/>
+                <geometry>
+                    <sphere radius="${raio_roda_boba}"/>
+                </geometry>
+                <material name="cinza_claro"/>
+            </visual>
+            <collision>
+                <origin xyz="0 0 0" rpy="0 0 0"/>
+                <geometry>
+                    <sphere radius="${raio_roda_boba}"/>
+                </geometry>
+                <surface>
+                    <friction>
+                        <ode>
+                            <mu>0.0</mu>
+                            <mu2>0.0</mu2>
+                            <slip1>1.0</slip1>
+                            <slip2>1.0</slip2>
+                        </ode>
+                    </friction>
+                    <contact>
+                        <ode>
+                            <soft_cfm>0</soft_cfm>
+                            <soft_erp>0.2</soft_erp>
+                            <kp>1e+13</kp>
+                            <kd>1</kd>
+                            <max_vel>0.01</max_vel>
+                            <min_depth>0.001</min_depth>
+                        </ode>
+                    </contact>
+                </surface>
+            </collision>
+            <inertial>
+                <origin xyz="0 0 0" rpy="0 0 0"/>
+                <mass value="${massa_roda_boba}"/>
+                <inertia ixx="${(2/5) * massa_roda_boba * (raio_roda_boba*raio_roda_boba)}" ixy="0.0" ixz="0.0" iyy="${(2/5) * massa_roda_boba * (raio_roda_boba*raio_roda_boba)}" iyz="0.0" izz="${(2/5) * massa_roda_boba * (raio_roda_boba*raio_roda_boba)}"/>
+            </inertial>
+        </link>
+        <joint name="${prefix}_roda_boba_junta" type="fixed">
+            <parent link="${parent}"/>
+            <child link="${prefix}_roda_boba_link"/>
+            <origin xyz="${x_offset} ${y_offset} ${z_offset}" rpy="0 0 0"/>
+        </joint>
+        <gazebo reference="${prefix}_roda_boba_link">
+            <material>Gazebo/DarkGrey</material>
+            <mu1>0.0</mu1>
+            <mu2>0.0</mu2>
+            <kp>1000000.0</kp>
+            <kd>10.0</kd>
+            <selfCollide>false</selfCollide>
+        </gazebo>
+    </xacro:macro>
+</robot>
